File: BMS_display_adapter_PCB/bms.kicad_pcb (KiCad board)
At the start: 2 copper layers, 313 x 211 mm, 66 parts, among them J1 55.5V, J10 22.2V, J11 18.5V, J12 14.8V, J13 11.1V, J14 7.4V, J15 3.7V, J16 0V, J17 Conn_01x02_Female, J18 Conn_01x02_Female, J19 Conn_01x02_Female, J2 51.8V, J20 Conn_01x02_Female, J21 Conn_01x02_Female, J22 Conn_01x02_Female, J23 Conn_01x02_Female, J24 Conn_01x02_Female, J25 Conn_01x02_Female, J26 Conn_01x02_Female, J27 Conn_01x02_Female, J28 Conn_01x02_Female, J29 Conn_01x02_Female, J3 48.1V, J30 Conn_01x02_Female, J31 Conn_01x02_Female, J32 Conn_01x18_Female, J33 Display Sense, J34 Conn_01x02_Female, J35 12V, J36 Conn_01x03_Male, J37 Pack -, J38 Conn_01x02_Female, J39 Batt input, J4 44.4V, J40 Conn_01x02_Female, J41 Conn_01x02_Female, J42 12v, J43 12v, J44 Conn_01x02_Female, J5 40.7V, J6 37V, J7 33.3V, J8 29.6V, J9 25.9V, M1 Fan

Commit message: work
Parts:
- added J45: Conn_01x01_Male, BMS:B2A-PCB, F.Cu at (-37.5, 167.5)
- added J46: Conn_01x01_Male, BMS:B2A-PCB, F.Cu at (-37.5, 179.3)
- added J47: Conn_01x01_Male, BMS:B2A-PCB, F.Cu at (-21.1, 167.5)
- added J48: Conn_01x01_Male, BMS:B2A-PCB, F.Cu at (-37.5, 191.1)
- added J49: Conn_01x01_Male, BMS:B2A-PCB, F.Cu at (-21.1, 179.3)
- added J50: Conn_01x01_Male, BMS:B2A-PCB, F.Cu at (-4.78, 167.5)
- added J51: Conn_01x01_Male, BMS:B2A-PCB, F.Cu at (-37.5, 202.9)
- added J52: Conn_01x01_Male, BMS:B2A-PCB, F.Cu at (-21.1, 191.1)
- added J53: Conn_01x01_Male, BMS:B2A-PCB, F.Cu at (-4.78, 179.3)
- added J54: Conn_01x01_Male, BMS:B2A-PCB, F.Cu at (11.6, 167.5)
- added J55: Conn_01x01_Male, BMS:B2A-PCB, F.Cu at (-21.1, 202.9)
- added J56: Conn_01x01_Male, BMS:B2A-PCB, F.Cu at (-4.78, 191.1)
- added J57: Conn_01x01_Male, BMS:B2A-PCB, F.Cu at (11.6, 179.3)
- added J58: Conn_01x01_Male, BMS:B2A-PCB, F.Cu at (27.9, 167.5)
- added J59: Conn_01x01_Male, BMS:B2A-PCB, F.Cu at (447.0, 174.0)
- added J60: Conn_01x01_Male, BMS:B2A-PCB, F.Cu at (11.6, 191.1)

Commit message: moving displays to make room for lugs
Parts:
- J45, J46, J47, J48, J49, J50, J51, J52, J53, J54, J55, J56, J57, J58, J59, J60: footprint BMS:B2A-PCB -> BMS:B4A-PCB
- moved J59 324.8 mm to (125.8, 222.0)
- moved J55 235.0 mm to (208.5, 253.0)
- moved J57 199.8 mm to (206.8, 222.0), turned to 90 degrees
- moved J45 185.7 mm to (117.5, 269.8)
- moved J46 185.7 mm to (117.5, 281.6)
- moved J47 185.7 mm to (133.9, 269.8)
- moved J48 185.7 mm to (117.5, 293.4)
- moved J49 185.7 mm to (133.9, 281.6)
- moved J50 185.7 mm to (150.2, 269.8)
- moved J52 185.7 mm to (133.9, 293.4)
- moved J53 185.7 mm to (150.2, 281.6)
- moved J54 185.7 mm to (166.6, 269.8)
- moved J56 185.7 mm to (150.2, 293.4)
- moved J58 148.7 mm to (166.2, 222.0), turned to 90 degrees
- moved J51 88.9 mm to (38.2, 249.5)
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Routing:
- net Net-(F8-Pad1): track 509.8 -> 254.9 mm
- net Net-(F7-Pad1): track 454.8 -> 227.4 mm
- net Net-(F9-Pad1): track 447.4 -> 223.7 mm
- net Net-(F6-Pad1): track 371.9 -> 186.0 mm
- net Net-(F10-Pad1): track 350.0 -> 175.0 mm
- net Net-(F14-Pad1): track 266.2 -> 99.1 mm
- net Net-(F5-Pad1): track 300.0 -> 150.0 mm
- net Net-(F15-Pad1): track 260.7 -> 124.4 mm
- net Earth: track 259.6 -> 129.8 mm
- net Net-(F11-Pad1): track 255.6 -> 127.8 mm
- net Net-(F1-Pad1): track 241.5 -> 121.3 mm
- net Net-(F4-Pad1): track 232.6 -> 116.3 mm
- net Net-(F2-Pad1): track 179.2 -> 89.6 mm
- net Net-(F13-Pad1): track 157.7 -> 75.6 mm
- net Net-(F12-Pad1): track 119.8 -> 59.9 mm
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- removed copper zone on B.Cu, net Earth
- removed copper zone on B.Cu, net Net-(F1-Pad1)
- removed copper zone on B.Cu, net Net-(F10-Pad1)
- removed copper zone on B.Cu, net Net-(F11-Pad1)
- removed copper zone on B.Cu, net Net-(F12-Pad1)
- removed copper zone on B.Cu, net Net-(F13-Pad1)
- removed copper zone on B.Cu, net Net-(F14-Pad1)
- removed copper zone on B.Cu, net Net-(F15-Pad1)
- removed copper zone on B.Cu, net Net-(F2-Pad1)
- removed copper zone on B.Cu, net Net-(F3-Pad1)
- removed copper zone on B.Cu, net Net-(F4-Pad1)
- removed copper zone on B.Cu, net Net-(F5-Pad1)
- removed copper zone on B.Cu, net Net-(F6-Pad1)
- removed copper zone on B.Cu, net Net-(F7-Pad1)
- removed copper zone on B.Cu, net Net-(F8-Pad1)
- removed copper zone on B.Cu, net Net-(F9-Pad1)

Commit message: redrawing planes
Parts:
- moved J51 362.0 mm to (323.8, 27.0), turned to 90 degrees
- moved J52 344.5 mm to (352.2, 27.0), turned to 90 degrees
- moved J48 279.3 mm to (201.5, 27.0), turned to 90 degrees
- moved J49 276.6 mm to (242.0, 27.0), turned to 90 degrees
- moved J50 276.6 mm to (282.8, 27.0), turned to 90 degrees
- moved J46 254.6 mm to (120.0, 27.0), turned to 90 degrees
- moved J45 245.2 mm to (81.2, 27.2), turned to 90 degrees
- moved J47 244.2 mm to (160.8, 27.0), turned to 90 degrees
- moved J53 215.2 mm to (357.0, 222.0), turned to 90 degrees
- moved J54 169.3 mm to (329.0, 222.0), turned to 90 degrees
- moved J56 120.9 mm to (247.8, 222.0), turned to 90 degrees
- moved J55 85.6 mm to (288.2, 222.0), turned to 90 degrees
- moved F8 17.2 mm to (366.5, 33.2)
- moved F9 13.8 mm to (368.2, 215.8)

Commit message: footprint updates
Parts:
- J1, J10, J11, J12, J13, J14, J15, J16, J2, J3, J4, J5, J6, J7, J8, J9: footprint BMS:m4_hole -> 1048:hole
- moved F8 1.75 mm to (368.2, 33.2)
- moved M1 0.57 mm to (179.2, 142.2)
- moved F1 0.50 mm to (72.8, 33.2)
Routing:
- net Net-(F8-Pad1): track 254.9 -> 528.8 mm
- net Net-(F9-Pad1): track 223.7 -> 460.4 mm
- net Net-(F7-Pad1): track 227.4 -> 462.2 mm
- net Net-(F6-Pad1): track 186.0 -> 389.1 mm
- net Net-(F10-Pad1): track 175.0 -> 371.5 mm
- net Net-(F5-Pad1): track 150.0 -> 319.0 mm
- net Net-(F11-Pad1): track 127.8 -> 277.1 mm
- net Earth: track 129.8 -> 268.6 mm
- net Net-(F4-Pad1): track 116.3 -> 249.1 mm
- net Net-(F15-Pad1): track 124.4 -> 248.9 mm
- net Net-(F1-Pad1): track 121.3 -> 242.6 mm
- net Net-(F14-Pad1): track 99.1 -> 190.7 mm
- net Net-(F2-Pad1): track 89.6 -> 179.3 mm
- net Net-(F13-Pad1): track 75.6 -> 150.9 mm
- net Net-(F3-Pad1): track 40.8 -> 86.4 mm
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- added copper zone on B.Cu, net Earth
- added copper zone on B.Cu, net Net-(F1-Pad1)
- added copper zone on B.Cu, net Net-(F10-Pad1)
- added copper zone on B.Cu, net Net-(F11-Pad1)
- added copper zone on B.Cu, net Net-(F12-Pad1)
- added copper zone on B.Cu, net Net-(F13-Pad1)
- added copper zone on B.Cu, net Net-(F14-Pad1)
- added copper zone on B.Cu, net Net-(F15-Pad1)
- added copper zone on B.Cu, net Net-(F2-Pad1)
- added copper zone on B.Cu, net Net-(F3-Pad1)
- added copper zone on B.Cu, net Net-(F4-Pad1)
- added copper zone on B.Cu, net Net-(F5-Pad1)
- added copper zone on B.Cu, net Net-(F6-Pad1)
- added copper zone on B.Cu, net Net-(F7-Pad1)
- added copper zone on B.Cu, net Net-(F8-Pad1)
- added copper zone on B.Cu, net Net-(F9-Pad1)
Other:
- board text added: "V1.2 by Vinnie Marco"
- board text removed: "V1.1 by Vinnie Marco"

Commit message: V1.2 Release
Parts:
- added F17: Fuse, BMS:Fuse, F.Cu at (72.8, 215.8)
- moved J52 5.00 mm to (357.2, 27.0)
- moved J59 1.50 mm to (124.2, 222.0)
- moved J46 1.25 mm to (118.8, 27.0)
- moved J47 1.25 mm to (159.5, 27.0)
- moved J48 1.25 mm to (200.2, 27.0)
- moved J49 1.25 mm to (240.8, 27.0)
- moved J50 1.25 mm to (281.5, 27.0)
- moved J54 1.25 mm to (327.8, 222.0)
- moved J55 1.25 mm to (287.0, 222.0)
- moved J56 1.25 mm to (246.5, 222.0)
- moved J57 1.25 mm to (205.5, 222.0)
- moved J58 1.25 mm to (165.0, 222.0)
- moved J60 1.25 mm to (83.8, 222.0)
- moved J51 1.00 mm to (322.8, 27.0)
- moved J53 0.25 mm to (357.2, 222.0)
Routing:
- net Earth: track 268.6 -> 283.8 mm
- net Net-(F13-Pad1): track 150.9 -> 144.3 mm
Other:
- board text added: "1x 250mA (F16) 1x 12V, 40mm fan 16x 3A Fuse (F0-F15) 1x XP Power - SRH05S12 1x 0-99V Display, Adafruit - 705 48x Pin headers - 0.1" male headers 19x Jumper block - 0.1" jumper block 15x 2.6-30V Display, Seeed - 114990163 15x B4A-PCB Lugsdirect"
- board text added: "F0"
- board text removed: "1x 250mA (F16) 1x 12V, 40mm fan 15x 3A Fuse (F1-F15) 1x XP Power - SRH05S12 1x 0-99V Display, Adafruit - 705 48x Pin headers - 0.1" male headers 19x Jumper block - 0.1" jumper block 15x 2.6-30V Display, Seeed - 114990163"
