File: BMS_display_adapter_PCB/bms.kicad_pcb (KiCad board)
At the start: 2 copper layers, 313 x 211 mm, 83 parts, among them J1 55.5V, J10 22.2V, J11 18.5V, J12 14.8V, J13 11.1V, J14 7.4V, J15 3.7V, J16 0V, J17 Conn_01x02_Female, J18 Conn_01x02_Female, J19 Conn_01x02_Female, J2 51.8V, J20 Conn_01x02_Female, J21 Conn_01x02_Female, J22 Conn_01x02_Female, J23 Conn_01x02_Female, J24 Conn_01x02_Female, J25 Conn_01x02_Female, J26 Conn_01x02_Female, J27 Conn_01x02_Female, J28 Conn_01x02_Female, J29 Conn_01x02_Female, J3 48.1V, J30 Conn_01x02_Female, J31 Conn_01x02_Female, J32 Conn_01x18_Female, J33 Display Sense, J34 Conn_01x02_Female, J35 12V, J36 Conn_01x03_Male, J37 Pack -, J38 Conn_01x02_Female, J39 Batt input, J4 44.4V, J40 Conn_01x02_Female, J41 Conn_01x02_Female, J42 12v, J43 12v, J44 Conn_01x02_Female, J45 Conn_01x01_Male, J46 Conn_01x01_Male, J47 Conn_01x01_Male, J48 Conn_01x01_Male, J49 Conn_01x01_Male, J5 40.7V, J50 Conn_01x01_Male, J51 Conn_01x01_Male, J52 Conn_01x01_Male, J53 Conn_01x01_Male, J54 Conn_01x01_Male, J55 Conn_01x01_Male, J56 Conn_01x01_Male, J57 Conn_01x01_Male, J58 Conn_01x01_Male, J59 Conn_01x01_Male, J6 37V, J60 Conn_01x01_Male, J7 33.3V, J8 29.6V, J9 25.9V, M1 Fan

Commit message: V1.2 Release
Parts:
- moved REF** 1.76 mm to (69.7, 124.5)
- moved REF** 1.72 mm to (371.0, 124.5)
Changed lines of the file:
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@@
   )
   (module MountingHole:MountingHole_4.3mm_M4_ISO7380_Pad locked (layer F.Cu)
-    (at 369.35 124)
+    (at 371 124.5)
     (descr "Mounting Hole 4.3mm, M4, ISO7380")
     (tags "mounting hole 4.3mm m4 iso7380")
@@
   )
   (module MountingHole:MountingHole_4.3mm_M4_ISO7380_Pad locked (layer F.Cu)
-    (at 68 124)
+    (at 69.7 124.45)
     (descr "Mounting Hole 4.3mm, M4, ISO7380")
     (tags "mounting hole 4.3mm m4 iso7380")
