File: BMS_display_adapter_PCB/bms.kicad_pcb (KiCad board)
At the start: 2 copper layers, 313 x 211 mm, 83 parts, among them J1 55.5V, J10 22.2V, J11 18.5V, J12 14.8V, J13 11.1V, J14 7.4V, J15 3.7V, J16 0V, J17 Conn_01x02_Female, J18 Conn_01x02_Female, J19 Conn_01x02_Female, J2 51.8V, J20 Conn_01x02_Female, J21 Conn_01x02_Female, J22 Conn_01x02_Female, J23 Conn_01x02_Female, J24 Conn_01x02_Female, J25 Conn_01x02_Female, J26 Conn_01x02_Female, J27 Conn_01x02_Female, J28 Conn_01x02_Female, J29 Conn_01x02_Female, J3 48.1V, J30 Conn_01x02_Female, J31 Conn_01x02_Female, J32 Conn_01x18_Female, J33 Display Sense, J34 Conn_01x02_Female, J35 12V, J36 Conn_01x03_Male, J37 Pack -, J38 Conn_01x02_Female, J39 Batt input, J4 44.4V, J40 Conn_01x02_Female, J41 Conn_01x02_Female, J42 12v, J43 12v, J44 Conn_01x02_Female, J45 Conn_01x01_Male, J46 Conn_01x01_Male, J47 Conn_01x01_Male, J48 Conn_01x01_Male, J49 Conn_01x01_Male, J5 40.7V, J50 Conn_01x01_Male, J51 Conn_01x01_Male, J52 Conn_01x01_Male, J53 Conn_01x01_Male, J54 Conn_01x01_Male, J55 Conn_01x01_Male, J56 Conn_01x01_Male, J57 Conn_01x01_Male, J58 Conn_01x01_Male, J59 Conn_01x01_Male, J6 37V, J60 Conn_01x01_Male, J7 33.3V, J8 29.6V, J9 25.9V, M1 Fan

Commit message: V1.3 Release
Other:
- board text added: "V1.3 by Vinnie Marco"
- board text removed: "V1.2 by Vinnie Marco"
Changed lines of the file:
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@@
   (general
     (thickness 1.6)
-    (drawings 1880)
+    (drawings 1884)
     (tracks 301)
     (zones 0)
@@
     (36 B.SilkS user)
     (37 F.SilkS user)
-    (38 B.Mask user)
-    (39 F.Mask user)
+    (38 B.Mask user hide)
+    (39 F.Mask user hide)
     (40 Dwgs.User user hide)
     (41 Cmts.User user hide)
@@
       (effects (font (size 0.7 0.7) (thickness 0.175)) (justify mirror))
     )
-    (fp_text user BAT1 (at 68.5 127.5) (layer B.SilkS)
+    (fp_text user BAT1 (at 68.5 122.75) (layer B.SilkS)
       (effects (font (size 0.7 0.7) (thickness 0.175)) (justify mirror))
     )
@@
       (effects (font (size 0.7 0.7) (thickness 0.175)))
     )
-    (fp_text user BAT1 (at 68.5 127.5) (layer F.SilkS)
+    (fp_text user BAT1 (at 68.5 122.75) (layer F.SilkS)
       (effects (font (size 0.7 0.7) (thickness 0.175)))
     )
@@
     )
   )
+  (module BMS:pack_voltmeter locked (layer F.Cu)
+    (at 85 124.571999 90)
+    (fp_text reference REF** (at 0.5 0 90) (layer F.SilkS) hide
+      (effects (font (size 1 1) (thickness 0.15)))
+    )
+    (fp_text value pack_voltmeter (at 0 -0.5 90) (layer F.Fab)
+      (effects (font (size 1 1) (thickness 0.15)))
+    )
+    (fp_line (start 2.5 7.25) (end 11.5 7.25) (layer Edge.Cuts) (width 0.12))
+    (fp_line (start -2.75 7.5) (end -11.75 7.5) (layer B.SilkS) (width 0.15))
+    (fp_line (start -2.75 8.75) (end -2.75 7.5) (layer B.SilkS) (width 0.15))
+    (fp_line (start 2.75 8.75) (end -2.75 8.75) (layer B.SilkS) (width 0.15))
+    (fp_line (start 2.75 7.5) (end 2.75 8.75) (layer B.SilkS) (width 0.15))
+    (fp_line (start 11.75 7.5) (end 2.75 7.5) (layer B.SilkS) (width 0.15))
+    (fp_line (start 2.75 7.5) (end 11.75 7.5) (layer F.SilkS) (width 0.15))
+    (fp_line (start -2.75 7.5) (end -11.75 7.5) (layer F.SilkS) (width 0.15))
+    (fp_line (start 2.75 8.75) (end 2.75 7.5) (layer F.SilkS) (width 0.15))
+    (fp_line (start -2.75 8.75) (end 2.75 8.75) (layer F.SilkS) (width 0.15))
+    (fp_line (start -2.75 7.5) (end -2.75 8.75) (layer F.SilkS) (width 0.15))
+    (fp_line (start 2.5 8.5) (end 2.5 7.25) (layer Edge.Cuts) (width 0.15))
+    (fp_line (start -2.5 8.5) (end 2.5 8.5) (layer Edge.Cuts) (width 0.15))
+    (fp_line (start -2.5 7.25) (end -2.5 8.5) (layer Edge.Cuts) (width 0.15))
+    (fp_line (start 11.75 -7.5) (end -11.75 -7.5) (layer B.SilkS) (width 0.15))
+    (fp_line (start 11.75 -2.5) (end 11.75 -7.5) (layer B.SilkS) (width 0.15))
+    (fp_line (start 16.25 -2.5) (end 11.75 -2.5) (layer B.SilkS) (width 0.15))
+    (fp_line (start 16.25 2.5) (end 16.25 -2.5) (layer B.SilkS) (width 0.15))
+    (fp_line (start 11.75 2.5) (end 16.25 2.5) (layer B.SilkS) (width 0.15))
+    (fp_line (start 11.75 7.5) (end 11.75 2.5) (layer B.SilkS) (width 0.15))
+    (fp_line (start -11.75 2.5) (end -11.75 7.5) (layer B.SilkS) (width 0.15))
+    (fp_line (start -16.25 2.5) (end -11.75 2.5) (layer B.SilkS) (width 0.15))
+    (fp_line (start -16.25 -2.5) (end -16.25 2.5) (layer B.SilkS) (width 0.15))
+    (fp_line (start -11.75 -2.5) (end -16.25 -2.5) (layer B.SilkS) (width 0.15))
+    (fp_line (start -11.75 -7.5) (end -11.75 -2.5) (layer B.SilkS) (width 0.15))
+    (fp_line (start 11.75 -2.5) (end 11.75 -7.5) (layer F.SilkS) (width 0.15))
+    (fp_line (start 11.75 2.5) (end 11.75 7.5) (layer F.SilkS) (width 0.15))
+    (fp_line (start 16.25 2.5) (end 11.75 2.5) (layer F.SilkS) (width 0.15))
+    (fp_line (start 16.25 -2.5) (end 16.25 2.5) (layer F.SilkS) (width 0.15))
+    (fp_line (start 11.75 -2.5) (end 16.25 -2.5) (layer F.SilkS) (width 0.15))
+    (fp_line (start -11.75 -2.5) (end -11.75 -7.5) (layer F.SilkS) (width 0.15))
+    (fp_line (start -11.75 2.5) (end -11.75 7.5) (layer F.SilkS) (width 0.15))
+    (fp_line (start -16.25 2.5) (end -11.75 2.5) (layer F.SilkS) (width 0.15))
+    (fp_line (start -16.25 -2.5) (end -16.25 2.5) (layer F.SilkS) (width 0.15))
+    (fp_line (start -11.75 -2.5) (end -16.25 -2.5) (layer F.SilkS) (width 0.15))
+    (fp_line (start 11.75 -7.5) (end -11.75 -7.5) (layer F.SilkS) (width 0.15))
+    (fp_line (start -11.5 7.25) (end -11.5 0.25) (layer Edge.Cuts) (width 0.12))
+    (fp_line (start 11.5 7.25) (end 11.5 -7.25) (layer Edge.Cuts) (width 0.12))
+    (fp_line (start -11.5 0.25) (end -11.5 -7.25) (layer Edge.Cuts) (width 0.12))
+    (fp_line (start -11.5 7.25) (end -2.5 7.25) (layer Edge.Cuts) (width 0.12))
+    (fp_line (start 11.5 -7.25) (end -11.5 -7.25) (layer Edge.Cuts) (width 0.12))
+    (pad "" thru_hole circle (at 14 0 90) (size 3.5 3.5) (drill 2) (layers *.Cu *.Mask))
+    (pad "" thru_hole circle (at -14 0 90) (size 3.5 3.5) (drill 2) (layers *.Cu *.Mask))
+    (model "${KIPRJMOD}/3D Models/LED DC 0-100V Digital Voltmeter Panel Meter.STEP"
+      (offset (xyz 0 0 4.5))
+      (scale (xyz 1 1.4 1))
+      (rotate (xyz 0 0 0))
+    )
+  )
   (module BMS:Fuse locked (layer F.Cu)
     (at 105 33.25 270)
@@
     )
   )
-  (module BMS:pack_voltmeter locked (layer F.Cu)
-    (at 85 124.571999 90)
-    (fp_text reference REF** (at 0.5 0 90) (layer F.SilkS) hide
-      (effects (font (size 1 1) (thickness 0.15)))
-    )
-    (fp_text value pack_voltmeter (at 0 -0.5 90) (layer F.Fab)
-      (effects (font (size 1 1) (thickness 0.15)))
-    )
-    (fp_line (start 11.75 -7.5) (end -11.75 -7.5) (layer B.SilkS) (width 0.15))
-    (fp_line (start 11.75 -2.5) (end 11.75 -7.5) (layer B.SilkS) (width 0.15))
-    (fp_line (start 16.25 -2.5) (end 11.75 -2.5) (layer B.SilkS) (width 0.15))
-    (fp_line (start 16.25 2.5) (end 16.25 -2.5) (layer B.SilkS) (width 0.15))
-    (fp_line (start 11.75 2.5) (end 16.25 2.5) (layer B.SilkS) (width 0.15))
-    (fp_line (start 11.75 7.5) (end 11.75 2.5) (layer B.SilkS) (width 0.15))
-    (fp_line (start -11.75 7.5) (end 11.75 7.5) (layer B.SilkS) (width 0.15))
-    (fp_line (start -11.75 2.5) (end -11.75 7.5) (layer B.SilkS) (width 0.15))
-    (fp_line (start -16.25 2.5) (end -11.75 2.5) (layer B.SilkS) (width 0.15))
-    (fp_line (start -16.25 -2.5) (end -16.25 2.5) (layer B.SilkS) (width 0.15))
-    (fp_line (start -11.75 -2.5) (end -16.25 -2.5) (layer B.SilkS) (width 0.15))
-    (fp_line (start -11.75 -7.5) (end -11.75 -2.5) (layer B.SilkS) (width 0.15))
-    (fp_line (start 11.75 -2.5) (end 11.75 -7.5) (layer F.SilkS) (width 0.15))
-    (fp_line (start 11.75 2.5) (end 11.75 7.5) (layer F.SilkS) (width 0.15))
-    (fp_line (start 16.25 2.5) (end 11.75 2.5) (layer F.SilkS) (width 0.15))
-    (fp_line (start 16.25 -2.5) (end 16.25 2.5) (layer F.SilkS) (width 0.15))
-    (fp_line (start 11.75 -2.5) (end 16.25 -2.5) (layer F.SilkS) (width 0.15))
-    (fp_line (start -11.75 -2.5) (end -11.75 -7.5) (layer F.SilkS) (width 0.15))
-    (fp_line (start -11.75 2.5) (end -11.75 7.5) (layer F.SilkS) (width 0.15))
-    (fp_line (start -16.25 2.5) (end -11.75 2.5) (layer F.SilkS) (width 0.15))
-    (fp_line (start -16.25 -2.5) (end -16.25 2.5) (layer F.SilkS) (width 0.15))
-    (fp_line (start -11.75 -2.5) (end -16.25 -2.5) (layer F.SilkS) (width 0.15))
-    (fp_line (start -11.75 7.5) (end 11.75 7.5) (layer F.SilkS) (width 0.15))
-    (fp_line (start 11.75 -7.5) (end -11.75 -7.5) (layer F.SilkS) (width 0.15))
-    (fp_line (start -11.5 7.25) (end -11.5 0.25) (layer Edge.Cuts) (width 0.12))
-    (fp_line (start 11.5 7.25) (end 11.5 -7.25) (layer Edge.Cuts) (width 0.12))
-    (fp_line (start -11.5 0.25) (end -11.5 -7.25) (layer Edge.Cuts) (width 0.12))
-    (fp_line (start -11.5 7.25) (end 11.5 7.25) (layer Edge.Cuts) (width 0.12))
-    (fp_line (start 11.5 -7.25) (end -11.5 -7.25) (layer Edge.Cuts) (width 0.12))
-    (pad "" thru_hole circle (at 14 0 90) (size 3.5 3.5) (drill 2) (layers *.Cu *.Mask))
-    (pad "" thru_hole circle (at -14 0 90) (size 3.5 3.5) (drill 2) (layers *.Cu *.Mask))
-    (model "${KIPRJMOD}/3D Models/LED DC 0-100V Digital Voltmeter Panel Meter.STEP"
-      (offset (xyz 0 0 4.5))
-      (scale (xyz 1 1.4 1))
-      (rotate (xyz 0 0 0))
-    )
-  )
   (module BMS:VoltMeter locked (layer F.Cu)
     (at 99 212 270)
@@
     (pad 1 thru_hole circle (at 0 0) (size 7.6 7.6) (drill 4.3) (layers *.Cu *.Mask))
   )
-  (gr_text "V1.2 by Vinnie Marco" (at 67.25 197 270) (layer B.SilkS)
+  (gr_text GND (at 100.99 173.73) (layer B.SilkS)
+    (effects (font (size 1 1) (thickness 0.25)) (justify mirror))
+  )
+  (gr_text GND (at 100.99 171.25) (layer B.SilkS)
+    (effects (font (size 1 1) (thickness 0.25)) (justify mirror))
+  )
+  (gr_text 12V (at 109.23 173.73) (layer B.SilkS)
+    (effects (font (size 1 1) (thickness 0.25)) (justify mirror))
+  )
+  (gr_text 12V (at 109.23 171.25) (layer B.SilkS)
+    (effects (font (size 1 1) (thickness 0.25)) (justify mirror))
+  )
+  (gr_text "V1.3 by Vinnie Marco" (at 67.26 196.97 270) (layer B.SilkS)
     (effects (font (size 2.5 2.5) (thickness 0.6)) (justify mirror))
   )
@@
     (effects (font (size 2.5 2.5) (thickness 0.6)))
   )
-  (gr_text "V1.2 by Vinnie Marco" (at 67.25 197 270) (layer F.SilkS)
+  (gr_text "V1.3 by Vinnie Marco" (at 67.25 197 270) (layer F.SilkS)
     (effects (font (size 2.5 2.5) (thickness 0.6)))
   )
@@
     (effects (font (size 4 4) (thickness 1)) (justify mirror))
   )
-  (gr_text "Pack Total" (at 96.25 124.25 90) (layer B.SilkS)
+  (gr_text "Pack Total" (at 96.82 124.57 90) (layer B.SilkS)
     (effects (font (size 4 4) (thickness 1)) (justify mirror))
   )
@@
     (effects (font (size 2.5 2.5) (thickness 0.5)))
   )
-  (gr_text "Pack Total" (at 96.25 124.5 90) (layer F.SilkS)
+  (gr_text "Pack Total" (at 96.82 124.82 90) (layer F.SilkS)
     (effects (font (size 4 4) (thickness 1)))
   )
