File: BMS_display_adapter_PCB/bms.sch (KiCad schematic (older format))
At the start: 61 parts, among them J1 55.5V, J10 22.2V, J11 18.5V, J12 14.8V, J13 11.1V, J14 7.4V, J15 3.7V, J16 0V, J17 Conn_01x02_Female, J18 Conn_01x02_Female, J19 Conn_01x02_Female, J2 51.8V, J20 Conn_01x02_Female, J21 Conn_01x02_Female, J22 Conn_01x02_Female, J23 Conn_01x02_Female, J24 Conn_01x02_Female, J25 Conn_01x02_Female, J26 Conn_01x02_Female, J27 Conn_01x02_Female, J28 Conn_01x02_Female, J29 Conn_01x02_Female, J3 48.1V, J30 Conn_01x02_Female, J31 Conn_01x02_Female, J32 Conn_01x18_Female, J33 Display Sense, J34 Conn_01x02_Female, J35 12V, J36 Conn_01x03_Male, J37 Pack -, J38 Conn_01x02_Female, J39 Batt input, J4 44.4V, J40 Conn_01x02_Female, J41 Conn_01x02_Female, J42 12v, J43 12v, J44 Conn_01x02_Female, J5 40.7V, J6 37V, J7 33.3V, J8 29.6V, J9 25.9V, M1 Fan

Commit message: work
Parts:
- added J45, J46, J47, J48, J49, J50, J51, J52, J53, J54, J55, J56, J57, J58, J59, J60: Conn_01x01_Male, BMS:B2A-PCB, symbol Connector:Conn_01x01_Male
Connections:
- net Earth: now also J60.1 (Pin_1)
- net at F15.1, F15.2, J15.1 (Pin_1)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: now also J59.1 (Pin_1)
- net at F14.1, F14.2, J14.1 (Pin_1)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: now also J58.1 (Pin_1)
- net at F13.1, F13.2, J13.1 (Pin_1)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: now also J57.1 (Pin_1)
- net at F12.1, F12.2, J12.1 (Pin_1)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: now also J56.1 (Pin_1)
- net at F11.1, F11.2, J11.1 (Pin_1)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: now also J55.1 (Pin_1)
- net at F10.1, F10.2, J10.1 (Pin_1)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: now also J54.1 (Pin_1)
- net at F9.1, F9.2, J24.2 (Pin_2)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: now also J53.1 (Pin_1)
- net at F8.1, F8.2, J23.2 (Pin_2)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: now also J52.1 (Pin_1)
- net at F7.1, F7.2, J22.2 (Pin_2)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: now also J51.1 (Pin_1)
- net at F6.1, F6.2, J21.2 (Pin_2)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: now also J50.1 (Pin_1)
- net at F5.1, F5.2, J20.2 (Pin_2)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: now also J49.1 (Pin_1)
- net at F4.1, F4.2, J19.2 (Pin_2)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: now also J48.1 (Pin_1)
- net at F3.1, F3.2, J18.2 (Pin_2)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: now also J47.1 (Pin_1)
- net at F2.1, F2.2, J17.2 (Pin_2)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: now also J46.1 (Pin_1)
- net at F1.1, F1.2, J1.1 (Pin_1)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: now also J45.1 (Pin_1)
Changed lines of the file:
@@
 	4050 3850 4050 3950
-Wire Wire Line
-	4050 3400 4050 3500
 Wire Wire Line
 	4050 2950 4050 3050
@@
 Wire Wire Line
 	7150 3800 7150 5050
+$Comp
+L Connector:Conn_01x01_Male J45
+U 1 1 5D4AB785
+P 4250 850
+F 0 "J45" H 4222 828 50  0000 R CNN
+F 1 "Conn_01x01_Male" H 4358 940 50  0001 C CNN
+F 2 "BMS:B2A-PCB" H 4250 850 50  0001 C CNN
+F 3 "~" H 4250 850 50  0001 C CNN
+	1    4250 850
+	-1   0    0    1
+$EndComp
+$Comp
+L Connector:Conn_01x01_Male J46
+U 1 1 5D4C1C37
+P 4250 1200
+F 0 "J46" H 4222 1178 50  0000 R CNN
+F 1 "Conn_01x01_Male" H 4358 1290 50  0001 C CNN
+F 2 "BMS:B2A-PCB" H 4250 1200 50  0001 C CNN
+F 3 "~" H 4250 1200 50  0001 C CNN
+	1    4250 1200
+	-1   0    0    1
+$EndComp
+$Comp
+L Connector:Conn_01x01_Male J47
+U 1 1 5D4C23E0
+P 4250 1600
+F 0 "J47" H 4222 1578 50  0000 R CNN
+F 1 "Conn_01x01_Male" H 4358 1690 50  0001 C CNN
+F 2 "BMS:B2A-PCB" H 4250 1600 50  0001 C CNN
+F 3 "~" H 4250 1600 50  0001 C CNN
+	1    4250 1600
+	-1   0    0    1
+$EndComp
+$Comp
+L Connector:Conn_01x01_Male J48
+U 1 1 5D4C2FA4
+P 4250 2050
+F 0 "J48" H 4222 2028 50  0000 R CNN
+F 1 "Conn_01x01_Male" H 4358 2140 50  0001 C CNN
+F 2 "BMS:B2A-PCB" H 4250 2050 50  0001 C CNN
+F 3 "~" H 4250 2050 50  0001 C CNN
+	1    4250 2050
+	-1   0    0    1
+$EndComp
+$Comp
+L Connector:Conn_01x01_Male J49
+U 1 1 5D4C34EC
+P 4250 2500
+F 0 "J49" H 4222 2478 50  0000 R CNN
+F 1 "Conn_01x01_Male" H 4358 2590 50  0001 C CNN
+F 2 "BMS:B2A-PCB" H 4250 2500 50  0001 C CNN
+F 3 "~" H 4250 2500 50  0001 C CNN
+	1    4250 2500
+	-1   0    0    1
+$EndComp
+$Comp
+L Connector:Conn_01x01_Male J50
+U 1 1 5D4C392E
+P 4250 2950
+F 0 "J50" H 4222 2928 50  0000 R CNN
+F 1 "Conn_01x01_Male" H 4358 3040 50  0001 C CNN
+F 2 "BMS:B2A-PCB" H 4250 2950 50  0001 C CNN
+F 3 "~" H 4250 2950 50  0001 C CNN
+	1    4250 2950
+	-1   0    0    1
+$EndComp
+Wire Wire Line
+	4050 3400 4050 3500
+$Comp
+L Connector:Conn_01x01_Male J51
+U 1 1 5D4C4732
+P 4250 3400
+F 0 "J51" H 4222 3378 50  0000 R CNN
+F 1 "Conn_01x01_Male" H 4358 3490 50  0001 C CNN
+F 2 "BMS:B2A-PCB" H 4250 3400 50  0001 C CNN
+F 3 "~" H 4250 3400 50  0001 C CNN
+	1    4250 3400
+	-1   0    0    1
+$EndComp
+$Comp
+L Connector:Conn_01x01_Male J52
+U 1 1 5D4C4B30
+P 4250 3850
+F 0 "J52" H 4222 3828 50  0000 R CNN
+F 1 "Conn_01x01_Male" H 4358 3940 50  0001 C CNN
+F 2 "BMS:B2A-PCB" H 4250 3850 50  0001 C CNN
+F 3 "~" H 4250 3850 50  0001 C CNN
+	1    4250 3850
+	-1   0    0    1
+$EndComp
+$Comp
+L Connector:Conn_01x01_Male J53
+U 1 1 5D4C4EC1
+P 4250 4300
+F 0 "J53" H 4222 4278 50  0000 R CNN
+F 1 "Conn_01x01_Male" H 4358 4390 50  0001 C CNN
+F 2 "BMS:B2A-PCB" H 4250 4300 50  0001 C CNN
+F 3 "~" H 4250 4300 50  0001 C CNN
+	1    4250 4300
+	-1   0    0    1
+$EndComp
+$Comp
+L Connector:Conn_01x01_Male J54
+U 1 1 5D4C525F
+P 4250 4750
+F 0 "J54" H 4222 4728 50  0000 R CNN
+F 1 "Conn_01x01_Male" H 4358 4840 50  0001 C CNN
+F 2 "BMS:B2A-PCB" H 4250 4750 50  0001 C CNN
+F 3 "~" H 4250 4750 50  0001 C CNN
+	1    4250 4750
+	-1   0    0    1
+$EndComp
+$Comp
+L Connector:Conn_01x01_Male J55
+U 1 1 5D4C5684
+P 4250 5200
+F 0 "J55" H 4222 5178 50  0000 R CNN
+F 1 "Conn_01x01_Male" H 4358 5290 50  0001 C CNN
+F 2 "BMS:B2A-PCB" H 4250 5200 50  0001 C CNN
+F 3 "~" H 4250 5200 50  0001 C CNN
+	1    4250 5200
+	-1   0    0    1
+$EndComp
+$Comp
+L Connector:Conn_01x01_Male J56
+U 1 1 5D4C5B37
+P 4250 5650
+F 0 "J56" H 4222 5628 50  0000 R CNN
+F 1 "Conn_01x01_Male" H 4358 5740 50  0001 C CNN
+F 2 "BMS:B2A-PCB" H 4250 5650 50  0001 C CNN
+F 3 "~" H 4250 5650 50  0001 C CNN
+	1    4250 5650
+	-1   0    0    1
+$EndComp
+$Comp
+L Connector:Conn_01x01_Male J57
+U 1 1 5D4C5F1A
+P 4250 6100
+F 0 "J57" H 4222 6078 50  0000 R CNN
+F 1 "Conn_01x01_Male" H 4358 6190 50  0001 C CNN
+F 2 "BMS:B2A-PCB" H 4250 6100 50  0001 C CNN
+F 3 "~" H 4250 6100 50  0001 C CNN
+	1    4250 6100
+	-1   0    0    1
+$EndComp
+$Comp
+L Connector:Conn_01x01_Male J58
+U 1 1 5D4C6179
+P 4250 6550
+F 0 "J58" H 4222 6528 50  0000 R CNN
+F 1 "Conn_01x01_Male" H 4358 6640 50  0001 C CNN
+F 2 "BMS:B2A-PCB" H 4250 6550 50  0001 C CNN
+F 3 "~" H 4250 6550 50  0001 C CNN
+	1    4250 6550
+	-1   0    0    1
+$EndComp
+$Comp
+L Connector:Conn_01x01_Male J59
+U 1 1 5D4C6501
+P 4250 7000
+F 0 "J59" H 4222 6978 50  0000 R CNN
+F 1 "Conn_01x01_Male" H 4358 7090 50  0001 C CNN
+F 2 "BMS:B2A-PCB" H 4250 7000 50  0001 C CNN
+F 3 "~" H 4250 7000 50  0001 C CNN
+	1    4250 7000
+	-1   0    0    1
+$EndComp
+$Comp
+L Connector:Conn_01x01_Male J60
+U 1 1 5D4C68FD
+P 4250 7450
+F 0 "J60" H 4222 7428 50  0000 R CNN
+F 1 "Conn_01x01_Male" H 4358 7540 50  0001 C CNN
+F 2 "BMS:B2A-PCB" H 4250 7450 50  0001 C CNN
+F 3 "~" H 4250 7450 50  0001 C CNN
+	1    4250 7450
+	-1   0    0    1
+$EndComp
 $EndSCHEMATC

Commit message: moving displays to make room for lugs
Parts:
- J45, J46, J47, J48, J49, J50, J51, J52, J53, J54, J55, J56, J57, J58, J59, J60: footprint BMS:B2A-PCB -> BMS:B4A-PCB
Changed lines of the file:
@@
 F 0 "J45" H 4222 828 50  0000 R CNN
 F 1 "Conn_01x01_Male" H 4358 940 50  0001 C CNN
-F 2 "BMS:B2A-PCB" H 4250 850 50  0001 C CNN
+F 2 "BMS:B4A-PCB" H 4250 850 50  0001 C CNN
 F 3 "~" H 4250 850 50  0001 C CNN
 	1    4250 850
@@
 F 0 "J46" H 4222 1178 50  0000 R CNN
 F 1 "Conn_01x01_Male" H 4358 1290 50  0001 C CNN
-F 2 "BMS:B2A-PCB" H 4250 1200 50  0001 C CNN
+F 2 "BMS:B4A-PCB" H 4250 1200 50  0001 C CNN
 F 3 "~" H 4250 1200 50  0001 C CNN
 	1    4250 1200
@@
 F 0 "J47" H 4222 1578 50  0000 R CNN
 F 1 "Conn_01x01_Male" H 4358 1690 50  0001 C CNN
-F 2 "BMS:B2A-PCB" H 4250 1600 50  0001 C CNN
+F 2 "BMS:B4A-PCB" H 4250 1600 50  0001 C CNN
 F 3 "~" H 4250 1600 50  0001 C CNN
 	1    4250 1600
@@
 F 0 "J48" H 4222 2028 50  0000 R CNN
 F 1 "Conn_01x01_Male" H 4358 2140 50  0001 C CNN
-F 2 "BMS:B2A-PCB" H 4250 2050 50  0001 C CNN
+F 2 "BMS:B4A-PCB" H 4250 2050 50  0001 C CNN
 F 3 "~" H 4250 2050 50  0001 C CNN
 	1    4250 2050
@@
 F 0 "J49" H 4222 2478 50  0000 R CNN
 F 1 "Conn_01x01_Male" H 4358 2590 50  0001 C CNN
-F 2 "BMS:B2A-PCB" H 4250 2500 50  0001 C CNN
+F 2 "BMS:B4A-PCB" H 4250 2500 50  0001 C CNN
 F 3 "~" H 4250 2500 50  0001 C CNN
 	1    4250 2500
@@
 F 0 "J50" H 4222 2928 50  0000 R CNN
 F 1 "Conn_01x01_Male" H 4358 3040 50  0001 C CNN
-F 2 "BMS:B2A-PCB" H 4250 2950 50  0001 C CNN
+F 2 "BMS:B4A-PCB" H 4250 2950 50  0001 C CNN
 F 3 "~" H 4250 2950 50  0001 C CNN
 	1    4250 2950
@@
 F 0 "J51" H 4222 3378 50  0000 R CNN
 F 1 "Conn_01x01_Male" H 4358 3490 50  0001 C CNN
-F 2 "BMS:B2A-PCB" H 4250 3400 50  0001 C CNN
+F 2 "BMS:B4A-PCB" H 4250 3400 50  0001 C CNN
 F 3 "~" H 4250 3400 50  0001 C CNN
 	1    4250 3400
@@
 F 0 "J52" H 4222 3828 50  0000 R CNN
 F 1 "Conn_01x01_Male" H 4358 3940 50  0001 C CNN
-F 2 "BMS:B2A-PCB" H 4250 3850 50  0001 C CNN
+F 2 "BMS:B4A-PCB" H 4250 3850 50  0001 C CNN
 F 3 "~" H 4250 3850 50  0001 C CNN
 	1    4250 3850
@@
 F 0 "J53" H 4222 4278 50  0000 R CNN
 F 1 "Conn_01x01_Male" H 4358 4390 50  0001 C CNN
-F 2 "BMS:B2A-PCB" H 4250 4300 50  0001 C CNN
+F 2 "BMS:B4A-PCB" H 4250 4300 50  0001 C CNN
 F 3 "~" H 4250 4300 50  0001 C CNN
 	1    4250 4300
@@
 F 0 "J54" H 4222 4728 50  0000 R CNN
 F 1 "Conn_01x01_Male" H 4358 4840 50  0001 C CNN
-F 2 "BMS:B2A-PCB" H 4250 4750 50  0001 C CNN
+F 2 "BMS:B4A-PCB" H 4250 4750 50  0001 C CNN
 F 3 "~" H 4250 4750 50  0001 C CNN
 	1    4250 4750
@@
 F 0 "J55" H 4222 5178 50  0000 R CNN
 F 1 "Conn_01x01_Male" H 4358 5290 50  0001 C CNN
-F 2 "BMS:B2A-PCB" H 4250 5200 50  0001 C CNN
+F 2 "BMS:B4A-PCB" H 4250 5200 50  0001 C CNN
 F 3 "~" H 4250 5200 50  0001 C CNN
 	1    4250 5200
@@
 F 0 "J56" H 4222 5628 50  0000 R CNN
 F 1 "Conn_01x01_Male" H 4358 5740 50  0001 C CNN
-F 2 "BMS:B2A-PCB" H 4250 5650 50  0001 C CNN
+F 2 "BMS:B4A-PCB" H 4250 5650 50  0001 C CNN
 F 3 "~" H 4250 5650 50  0001 C CNN
 	1    4250 5650
@@
 F 0 "J57" H 4222 6078 50  0000 R CNN
 F 1 "Conn_01x01_Male" H 4358 6190 50  0001 C CNN
-F 2 "BMS:B2A-PCB" H 4250 6100 50  0001 C CNN
+F 2 "BMS:B4A-PCB" H 4250 6100 50  0001 C CNN
 F 3 "~" H 4250 6100 50  0001 C CNN
 	1    4250 6100
@@
 F 0 "J58" H 4222 6528 50  0000 R CNN
 F 1 "Conn_01x01_Male" H 4358 6640 50  0001 C CNN
-F 2 "BMS:B2A-PCB" H 4250 6550 50  0001 C CNN
+F 2 "BMS:B4A-PCB" H 4250 6550 50  0001 C CNN
 F 3 "~" H 4250 6550 50  0001 C CNN
 	1    4250 6550
@@
 F 0 "J59" H 4222 6978 50  0000 R CNN
 F 1 "Conn_01x01_Male" H 4358 7090 50  0001 C CNN
-F 2 "BMS:B2A-PCB" H 4250 7000 50  0001 C CNN
+F 2 "BMS:B4A-PCB" H 4250 7000 50  0001 C CNN
 F 3 "~" H 4250 7000 50  0001 C CNN
 	1    4250 7000
@@
 F 0 "J60" H 4222 7428 50  0000 R CNN
 F 1 "Conn_01x01_Male" H 4358 7540 50  0001 C CNN
-F 2 "BMS:B2A-PCB" H 4250 7450 50  0001 C CNN
+F 2 "BMS:B4A-PCB" H 4250 7450 50  0001 C CNN
 F 3 "~" H 4250 7450 50  0001 C CNN
 	1    4250 7450

Commit message: footprint updates
Parts:
- J1, J10, J11, J12, J13, J14, J15, J16, J2, J3, J4, J5, J6, J7, J8, J9: footprint BMS:m4_hole -> 1048:hole
Changed lines of the file:
@@
 F 0 "J1" H 3750 750 50  0001 C CNN
 F 1 "55.5V" H 3700 750 50  0000 C CNN
-F 2 "BMS:m4_hole" H 3850 750 50  0001 C CNN
+F 2 "1048:hole" H 3850 750 50  0001 C CNN
 F 3 "~" H 3850 750 50  0001 C CNN
 	1    3850 750
@@
 F 0 "J2" H 3750 1200 50  0001 C CNN
 F 1 "51.8V" H 3700 1200 50  0000 C CNN
-F 2 "BMS:m4_hole" H 3850 1200 50  0001 C CNN
+F 2 "1048:hole" H 3850 1200 50  0001 C CNN
 F 3 "~" H 3850 1200 50  0001 C CNN
 	1    3850 1200
@@
 F 0 "J3" H 3750 1600 50  0001 C CNN
 F 1 "48.1V" H 3700 1600 50  0000 C CNN
-F 2 "BMS:m4_hole" H 3850 1600 50  0001 C CNN
+F 2 "1048:hole" H 3850 1600 50  0001 C CNN
 F 3 "~" H 3850 1600 50  0001 C CNN
 	1    3850 1600
@@
 F 0 "J4" H 3750 2050 50  0001 C CNN
 F 1 "44.4V" H 3700 2050 50  0000 C CNN
-F 2 "BMS:m4_hole" H 3850 2050 50  0001 C CNN
+F 2 "1048:hole" H 3850 2050 50  0001 C CNN
 F 3 "~" H 3850 2050 50  0001 C CNN
 	1    3850 2050
@@
 F 0 "J5" H 3750 2500 50  0001 C CNN
 F 1 "40.7V" H 3700 2500 50  0000 C CNN
-F 2 "BMS:m4_hole" H 3850 2500 50  0001 C CNN
+F 2 "1048:hole" H 3850 2500 50  0001 C CNN
 F 3 "~" H 3850 2500 50  0001 C CNN
 	1    3850 2500
@@
 F 0 "J7" H 3750 3400 50  0001 C CNN
 F 1 "33.3V" H 3700 3400 50  0000 C CNN
-F 2 "BMS:m4_hole" H 3850 3400 50  0001 C CNN
+F 2 "1048:hole" H 3850 3400 50  0001 C CNN
 F 3 "~" H 3850 3400 50  0001 C CNN
 	1    3850 3400
@@
 F 0 "J11" H 3750 5200 50  0001 C CNN
 F 1 "18.5V" H 3700 5200 50  0000 C CNN
-F 2 "BMS:m4_hole" H 3850 5200 50  0001 C CNN
+F 2 "1048:hole" H 3850 5200 50  0001 C CNN
 F 3 "~" H 3850 5200 50  0001 C CNN
 	1    3850 5200
@@
 F 0 "J13" H 3750 6100 50  0001 C CNN
 F 1 "11.1V" H 3700 6100 50  0000 C CNN
-F 2 "BMS:m4_hole" H 3850 6100 50  0001 C CNN
+F 2 "1048:hole" H 3850 6100 50  0001 C CNN
 F 3 "~" H 3850 6100 50  0001 C CNN
 	1    3850 6100
@@
 F 0 "J14" H 3750 6550 50  0001 C CNN
 F 1 "7.4V" H 3750 6550 50  0000 C CNN
-F 2 "BMS:m4_hole" H 3850 6550 50  0001 C CNN
+F 2 "1048:hole" H 3850 6550 50  0001 C CNN
 F 3 "~" H 3850 6550 50  0001 C CNN
 	1    3850 6550
@@
 F 0 "J15" H 3750 7000 50  0001 C CNN
 F 1 "3.7V" H 3750 7000 50  0000 C CNN
-F 2 "BMS:m4_hole" H 3850 7000 50  0001 C CNN
+F 2 "1048:hole" H 3850 7000 50  0001 C CNN
 F 3 "~" H 3850 7000 50  0001 C CNN
 	1    3850 7000
@@
 F 0 "J16" H 3750 7450 50  0001 C CNN
 F 1 "0V" H 3750 7450 50  0000 C CNN
-F 2 "BMS:m4_hole" H 3850 7450 50  0001 C CNN
+F 2 "1048:hole" H 3850 7450 50  0001 C CNN
 F 3 "~" H 3850 7450 50  0001 C CNN
 	1    3850 7450
@@
 F 0 "J12" H 3750 5650 50  0001 C CNN
 F 1 "14.8V" H 3700 5650 50  0000 C CNN
-F 2 "BMS:m4_hole" H 3850 5650 50  0001 C CNN
+F 2 "1048:hole" H 3850 5650 50  0001 C CNN
 F 3 "~" H 3850 5650 50  0001 C CNN
 	1    3850 5650
@@
 F 0 "J9" H 3750 4300 50  0001 C CNN
 F 1 "25.9V" H 3700 4300 50  0000 C CNN
-F 2 "BMS:m4_hole" H 3850 4300 50  0001 C CNN
+F 2 "1048:hole" H 3850 4300 50  0001 C CNN
 F 3 "~" H 3850 4300 50  0001 C CNN
 	1    3850 4300
@@
 F 0 "J8" H 3750 3850 50  0001 C CNN
 F 1 "29.6V" H 3700 3850 50  0000 C CNN
-F 2 "BMS:m4_hole" H 3850 3850 50  0001 C CNN
+F 2 "1048:hole" H 3850 3850 50  0001 C CNN
 F 3 "~" H 3850 3850 50  0001 C CNN
 	1    3850 3850
@@
 F 0 "J6" H 3750 2950 50  0001 C CNN
 F 1 "37V" H 3750 2950 50  0000 C CNN
-F 2 "BMS:m4_hole" H 3850 2950 50  0001 C CNN
+F 2 "1048:hole" H 3850 2950 50  0001 C CNN
 F 3 "~" H 3850 2950 50  0001 C CNN
 	1    3850 2950
@@
 F 0 "J10" H 3750 4750 50  0001 C CNN
 F 1 "22.2V" H 3700 4750 50  0000 C CNN
-F 2 "BMS:m4_hole" H 3850 4750 50  0001 C CNN
+F 2 "1048:hole" H 3850 4750 50  0001 C CNN
 F 3 "~" H 3850 4750 50  0001 C CNN
 	1    3850 4750

Commit message: V1.2 Release
Parts:
- added F17: Fuse, BMS:Fuse, symbol Device:Fuse
Connections:
- net Earth: now also F17.1, F17.2
Changed lines of the file:
@@
 	1    0    0    -1
 $EndComp
-Wire Wire Line
-	4050 7450 4050 7500
 $Comp
 L Connector:Conn_01x01_Male J16
@@
 Wire Wire Line
 	2200 4900 2200 5000
-Wire Wire Line
-	2200 7500 4050 7500
 Connection ~ 2200 5000
-Connection ~ 4050 7500
-Wire Wire Line
-	4050 7500 4050 7550
 Wire Wire Line
 	2200 5000 2200 7500
@@
 	-1   0    0    1
 $EndComp
+Wire Wire Line
+	4050 7450 4050 7500
+$Comp
+L Device:Fuse F17
+U 1 1 5D535347
+P 3100 7500
+F 0 "F17" V 2995 7500 50  0000 C CNN
+F 1 "Fuse" V 2994 7500 50  0001 C CNN
+F 2 "BMS:Fuse" V 3030 7500 50  0001 C CNN
+F 3 "~" H 3100 7500 50  0001 C CNN
+	1    3100 7500
+	0    1    1    0
+$EndComp
+Wire Wire Line
+	2200 7500 2900 7500
+Wire Wire Line
+	3250 7500 3300 7500
+Connection ~ 4050 7500
+Wire Wire Line
+	4050 7500 4050 7550
+Wire Wire Line
+	2900 7500 2900 7350
+Wire Wire Line
+	2900 7350 3300 7350
+Wire Wire Line
+	3300 7350 3300 7500
+Connection ~ 2900 7500
+Wire Wire Line
+	2900 7500 2950 7500
+Connection ~ 3300 7500
+Wire Wire Line
+	3300 7500 4050 7500
 $EndSCHEMATC
