File: 15s4p_PCB/15s4p_board.kicad_pcb (KiCad board)
At the start: 2 copper layers, 313 x 211 mm, 174 parts, among them J1 18.5V, J10 25.9V, J11 22.2V, J12 55.5V, J13 51.8V, J14 48.1V, J15 44.4V, J16 40.7V, J2 14.8V, J3 11.1V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

Commit message: V2.5 Release
updated standoff pads
Other:
- board text added: "V2.5 by Vinnie Marco"
- board text removed: "V2.4 by Vinnie Marco"
